Commit message: fix error optical frame in rtabmap

File: thesis_robot_modeling/urdf/thesis_robot_modeling.urdf (robot description, URDF)
Before this commit: robot thesis_robot_modeling, 8 links, 7 joints
Links:
- removed link realsense_link
- added link camera_link, mass 0.10349; collision mesh filename=package://thesis_robot_modeling/meshes/realsense_link.STL; visual mesh filename=package://thesis_robot_modeling/meshes/realsense_link.STL
Joints:
- joint realsense_joint: child realsense_link -> camera_link

File: thesis_robot_modeling/urdf/thesis_robot_modeling.urdf.xacro (robot description, xacro)
@@ -180,9 +180,9 @@
     <origin xyz="0.079 0.001 0.285" rpy="-1.57 0 -1.57" />
     <parent link="base_link" />
-    <child link="camera_link" />
+    <child link="realsense_link" />
     <axis xyz="0 0 0" />
     <safety_controller k_velocity="0" />
   </joint>
-  <link name="camera_link">
+  <link name="realsense_link">
     <inertial>
       <origin xyz="0 0 0" rpy="0 0 0" />
@@ -245,3 +245,38 @@
     </collision>
   </link>
+<joint name="camera_joint" type="fixed">
+    <origin xyz="0 0 0" rpy="0 0 0" />
+    <parent link="realsense_link" />
+    <child link="camera_link" />
+    <axis xyz="0 0 0" />
+  </joint>
+<link name="camera_link"/>
+<joint name="camera_depth_joint" type="fixed">
+    <origin xyz="0 0 0" rpy="0 0 0" />
+    <parent link="realsense_link" />
+    <child link="camera_depth_frame" />
+    <axis xyz="0 0 0" />
+  </joint>
+  <link name="camera_depth_frame"/>
+<joint name="camera_color_joint" type="fixed">
+    <origin xyz="0 0 0" rpy="0 0 0" />
+    <parent link="realsense_link" />
+    <child link="camera_color_frame" />
+    <axis xyz="0 0 0" />
+  </joint>
+  <link name="camera_color_frame"/>
+  <joint name="camera_depth_optical_joint" type="fixed">
+    <origin xyz="0 0 0" rpy="0 0 0" />
+    <parent link="realsense_link" />
+    <child link="camera_depth_optical_frame" />
+    <axis xyz="0 0 0" />
+  </joint>
+  <link name="camera_depth_optical_frame"/>
+<joint name="camera_color_optical_joint" type="fixed">
+    <origin xyz="0 0 0" rpy="0 0 0" />
+    <parent link="realsense_link" />
+    <child link="camera_color_optical_frame" />
+    <axis xyz="0 0 0" />
+  </joint>
+  <link name="camera_color_optical_frame"/>
 </robot>
