Commit message: nothing

File: thesis_robot_modeling/urdf/thesis_robot_modeling.urdf copy.xacro (robot description, xacro)
@@ -147,7 +147,7 @@
     <origin xyz="-0.01 0 0.335" rpy="0 0 3.14" />
     <parent link="base_link" />
-    <child link="rplidar_link" />
-  </joint>
-  <link name="rplidar_link">
+    <child link="lidar_link" />
+  </joint>
+  <link name="lidar_link">
     <inertial>
       <origin xyz="0 0 0" rpy="0 0 0" />
