Commit message: modified model

File: thesis_robot_modeling/urdf/thesis_robot_modeling.urdf.xacro (robot description, xacro)
@@ -9,5 +9,5 @@
     <parent link="base_footprint"/>
     <child link="base_link"/>
-    <origin xyz="0 0 0.1" rpy="0 0 1.57"/>
+    <origin xyz="0 0 0.1" rpy="0 0 3.14"/>
   </joint>
   <link name="base_link">
@@ -25,5 +25,5 @@
     </inertial>
     <visual>
-      <origin xyz="0 0 0" rpy="0 0 0" />
+      <origin xyz="0 0 0" rpy="0 0 -1.57" />
       <geometry>
         <mesh filename="package://thesis_robot_modeling/meshes/base_link.STL" />
@@ -34,5 +34,5 @@
     </visual>
     <collision>
-      <origin xyz="0 0 0" rpy="0 0 0" />
+      <origin xyz="0 0 0" rpy="0 0 -1.57" />
       <geometry>
         <mesh filename="package://thesis_robot_modeling/meshes/base_link.STL" />

Commit message: modified urdf model

File: thesis_robot_modeling/urdf/thesis_robot_modeling.urdf.xacro (robot description, xacro)
@@ -9,9 +9,8 @@
     <parent link="base_footprint"/>
     <child link="base_link"/>
-    <origin xyz="0 0 0.1" rpy="0 0 3.14"/>
+    <origin xyz="0 0 0.1" rpy="0 0 0"/>
   </joint>
   <link name="base_link">
     <inertial>
-      <!--origin xyz="0.00058448 0.32986 -0.021877" rpy="0 0 0" /-->
       <origin xyz="0 0 0" rpy="0 0 0"/>
       <mass value="2.1405"/>
@@ -25,5 +24,5 @@
     </inertial>
     <visual>
-      <origin xyz="0 0 0" rpy="0 0 -1.57" />
+      <origin xyz="-0.18 -0.2023 -0.182" rpy="1.57 0 1.57" />
       <geometry>
         <mesh filename="package://thesis_robot_modeling/meshes/base_link.STL" />
@@ -34,5 +33,5 @@
     </visual>
     <collision>
-      <origin xyz="0 0 0" rpy="0 0 -1.57" />
+      <origin xyz="0 0 0" rpy="0 0 0" />
       <geometry>
         <mesh filename="package://thesis_robot_modeling/meshes/base_link.STL" />
@@ -40,6 +39,6 @@
     </collision>
   </link>
-  <joint name="left_wheel_joint" type="continuous">
-    <origin xyz="0.17221 0.071027 0.045506" rpy="0 1.57 0" />
+  <joint name="left_wheel_joint" type="fixed">
+    <origin xyz="-0.071027 0.18221 -0.046496" rpy="-1.57 1.57 0" />
     <parent link="base_link" />
     <child link="left_wheel_link" />
@@ -76,6 +75,6 @@
     </collision>
   </link>
-  <joint name="right_wheel_joint" type="continuous">
-    <origin xyz="-0.17221 0.071027 0.045506" rpy="0 1.57 0" />
+  <joint name="right_wheel_joint" type="fixed">
+    <origin xyz="-0.071027 -0.18221 -0.046496" rpy="-1.57 1.57 0" />
     <parent link="base_link" />
     <child link="right_wheel_link" />
@@ -111,5 +110,5 @@
   </link>
   <joint name="caster_wheel_joint" type="fixed">
-    <origin xyz="0 -0.10103 0.015" rpy="-1.5708 0 1.5708" />
+    <origin xyz="0.10103 0 -0.077" rpy="-1.5708 0 0" />
     <parent link="base_link" />
     <child link="caster_wheel_link" />
@@ -146,5 +145,5 @@
   </link>
   <joint name="lidar_joint" type="fixed">
-    <origin xyz="0 0.01 0.785" rpy="0 0 1.57" />
+    <origin xyz="-0.01 0 0.335" rpy="0 0 0" />
     <parent link="base_link" />
     <child link="lidar_link" />
@@ -163,5 +162,5 @@
     </inertial>
     <visual>
-      <origin xyz="-0.01 0 -0.785" rpy="1.57 0 -1.57" />
+      <origin xyz="0.01 0 -0.785" rpy="1.57 0 1.57" />
       <geometry>
         <mesh filename="package://thesis_robot_modeling/meshes/lidar_link.STL" />
@@ -179,5 +178,5 @@
   </link>
   <joint name="realsense_joint" type="fixed">
-    <origin xyz="0.001 -0.079 0.73355" rpy="0 0 1.57" />
+    <origin xyz="0.079 0.001 0.285" rpy="0 0 0" />
     <parent link="base_link" />
     <child link="realsense_link" />
@@ -198,5 +197,5 @@
     </inertial>
     <visual>
-      <origin xyz="0.078 0 -0.735" rpy="1.57 0 -1.57" />
+      <origin xyz="-0.078 0 -0.735" rpy="1.57 0 1.57" />
       <geometry>
         <mesh filename="package://thesis_robot_modeling/meshes/realsense_link.STL" />
@@ -214,5 +213,5 @@
   </link>
   <joint name="imu_joint" type="fixed">
-    <origin xyz="-0.071997 -0.039397 0.41026" rpy="0 0 1.57" />
+    <origin xyz="0.039397 -0.071997 0.138" rpy="0 0 0" />
     <parent link="base_link" />
     <child link="imu_link" />
@@ -221,5 +220,5 @@
     <inertial>
       <origin xyz="0 0 0" rpy="0 0 0" />
-      <mass value="0.00064128" />
+      <mass value="0.00064128"/>
       <inertia
         ixx="1.1862E-08"
@@ -231,5 +230,5 @@
     </inertial>
     <visual>
-      <origin xyz="0.038 -0.0713 -0.415" rpy="1.57 0 -1.57" />
+      <origin xyz="-0.038 0.0713 -0.415" rpy="1.57 0 1.57" />
       <geometry>
         <mesh filename="package://thesis_robot_modeling/meshes/imu_link.STL" />

Commit message: modified on Jetson

File: thesis_robot_modeling/urdf/thesis_robot_modeling.urdf.xacro (robot description, xacro)
@@ -9,5 +9,5 @@
     <parent link="base_footprint"/>
     <child link="base_link"/>
-    <origin xyz="0 0 0.1" rpy="0 0 3.14"/>
+    <origin xyz="0 0 0.1" rpy="0 0 0"/>
   </joint>
   <link name="base_link">
@@ -25,5 +25,5 @@
     </inertial>
     <visual>
-      <origin xyz="0 0 0" rpy="0 0 -1.57" />
+      <origin xyz="0 0 0" rpy="0 0 0" />
       <geometry>
         <mesh filename="package://thesis_robot_modeling/meshes/base_link.STL" />
@@ -34,5 +34,5 @@
     </visual>
     <collision>
-      <origin xyz="0 0 0" rpy="0 0 -1.57" />
+      <origin xyz="0 0 0" rpy="0 0 0" />
       <geometry>
         <mesh filename="package://thesis_robot_modeling/meshes/base_link.STL" />

Commit message: create new branch for c heckpoint

File: thesis_robot_modeling/urdf/thesis_robot_modeling.urdf.xacro (robot description, xacro)
@@ -9,5 +9,5 @@
     <parent link="base_footprint"/>
     <child link="base_link"/>
-    <origin xyz="0 0 0.1" rpy="0 0 3.14"/>
+    <origin xyz="0 0 0.1" rpy="0 0 0"/>
   </joint>
   <link name="base_link">
@@ -145,5 +145,5 @@
   </link>
   <joint name="lidar_joint" type="fixed">
-    <origin xyz="-0.01 0 0.335" rpy="0 0 0" />
+    <origin xyz="-0.01 0 0.335" rpy="0 0 3.14" />
     <parent link="base_link" />
     <child link="lidar_link" />
@@ -162,5 +162,5 @@
     </inertial>
     <visual>
-      <origin xyz="0.01 0 -0.785" rpy="1.57 0 1.57" />
+      <origin xyz="-0.01 0 -0.785" rpy="1.57 0 -1.57" />
       <geometry>
         <mesh filename="package://thesis_robot_modeling/meshes/lidar_link.STL" />
@@ -171,5 +171,5 @@
     </visual>
     <collision>
-      <origin xyz="0 0 0" rpy="1.57 0 -1.57" />
+      <origin xyz="-0.01 0 -0.785" rpy="1.57 0 -1.57" />
       <geometry>
         <mesh filename="package://thesis_robot_modeling/meshes/lidar_link.STL" />
@@ -178,5 +178,5 @@
   </link>
   <joint name="realsense_joint" type="fixed">
-    <origin xyz="0.079 0.001 0.285" rpy="0 0 0" />
+    <origin xyz="0.079 0.001 0.285" rpy="-1.57 0 -1.57" />
     <parent link="base_link" />
     <child link="realsense_link" />
@@ -197,5 +197,5 @@
     </inertial>
     <visual>
-      <origin xyz="-0.078 0 -0.735" rpy="1.57 0 1.57" />
+      <origin xyz="0 0.735 -0.078" rpy="3.14 3.14 0" />
       <geometry>
         <mesh filename="package://thesis_robot_modeling/meshes/realsense_link.STL" />
@@ -206,5 +206,5 @@
     </visual>
     <collision>
-      <origin xyz="0 0 0" rpy="1.57 0 -1.57" />
+      <origin xyz="0 0.735 -0.078" rpy="3.14 3.14 0" />
       <geometry>
         <mesh filename="package://thesis_robot_modeling/meshes/realsense_link.STL" />
@@ -239,5 +239,5 @@
     </visual>
     <collision>
-      <origin xyz="0 0 0" rpy="0 0 0" />
+      <origin xyz="-0.038 0.0713 -0.415" rpy="1.57 0 1.57" />
       <geometry>
         <mesh filename="package://thesis_robot_modeling/meshes/imu_link.STL" />

Commit message: change version realsense ros to 2.2.22

File: thesis_robot_modeling/urdf/thesis_robot_modeling.urdf.xacro (robot description, xacro)
@@ -147,7 +147,7 @@
     <origin xyz="-0.01 0 0.335" rpy="0 0 3.14" />
     <parent link="base_link" />
-    <child link="lidar_link" />
-  </joint>
-  <link name="lidar_link">
+    <child link="rplidar_link" />
+  </joint>
+  <link name="rplidar_link">
     <inertial>
       <origin xyz="0 0 0" rpy="0 0 0" />
@@ -180,9 +180,9 @@
     <origin xyz="0.079 0.001 0.285" rpy="-1.57 0 -1.57" />
     <parent link="base_link" />
-    <child link="realsense_link" />
+    <child link="camera_link" />
     <axis xyz="0 0 0" />
     <safety_controller k_velocity="0" />
   </joint>
-  <link name="realsense_link">
+  <link name="camera_link">
     <inertial>
       <origin xyz="0 0 0" rpy="0 0 0" />

Commit message: config realsense ros just use necessary topic

File: thesis_robot_modeling/urdf/thesis_robot_modeling.urdf.xacro (robot description, xacro)
@@ -144,10 +144,10 @@
     </collision>
   </link>
-  <joint name="lidar_joint" type="fixed">
+  <joint name="rplidar_joint" type="fixed">
     <origin xyz="-0.01 0 0.335" rpy="0 0 3.14" />
     <parent link="base_link" />
-    <child link="rplidar_link" />
-  </joint>
-  <link name="rplidar_link">
+    <child link="lidar_link" />
+  </joint>
+  <link name="lidar_link">
     <inertial>
       <origin xyz="0 0 0" rpy="0 0 0" />

Commit message: sync to jetsonnano

File: thesis_robot_modeling/urdf/thesis_robot_modeling.urdf.xacro (robot description, xacro)
@@ -180,9 +180,9 @@
     <origin xyz="0.079 0.001 0.285" rpy="-1.57 0 -1.57" />
     <parent link="base_link" />
-    <child link="realsense_link" />
+    <child link="camera_link" />
     <axis xyz="0 0 0" />
     <safety_controller k_velocity="0" />
   </joint>
-  <link name="realsense_link">
+  <link name="camera_link">
     <inertial>
       <origin xyz="0 0 0" rpy="0 0 0" />

Commit message: add other slam

File: thesis_robot_modeling/urdf/thesis_robot_modeling.urdf.xacro (robot description, xacro)
@@ -180,9 +180,9 @@
     <origin xyz="0.079 0.001 0.285" rpy="-1.57 0 -1.57" />
     <parent link="base_link" />
-    <child link="camera_link" />
+    <child link="realsense_link" />
     <axis xyz="0 0 0" />
     <safety_controller k_velocity="0" />
   </joint>
-  <link name="camera_link">
+  <link name="realsense_link">
     <inertial>
       <origin xyz="0 0 0" rpy="0 0 0" />

Commit message: nothing

File: thesis_robot_modeling/urdf/thesis_robot_modeling.urdf.xacro (robot description, xacro)
@@ -144,37 +144,4 @@
     </collision>
   </link>
-  <joint name="rplidar_joint" type="fixed">
-    <origin xyz="-0.01 0 0.335" rpy="0 0 3.14" />
-    <parent link="base_link" />
-    <child link="lidar_link" />
-  </joint>
-  <link name="lidar_link">
-    <inertial>
-      <origin xyz="0 0 0" rpy="0 0 0" />
-      <mass value="0.021237" />
-      <inertia
-        ixx="0.00016144"
-        ixy="2.1931E-07"
-        ixz="-4.8964E-07"
-        iyy="0.00020117"
-        iyz="-2.029E-05"
-        izz="0.00010111" />
-    </inertial>
-    <visual>
-      <origin xyz="-0.01 0 -0.785" rpy="1.57 0 -1.57" />
-      <geometry>
-        <mesh filename="package://thesis_robot_modeling/meshes/lidar_link.STL" />
-      </geometry>
-      <material name="">
-        <color rgba="0.79216 0.81961 0.93333 1" />
-      </material>
-    </visual>
-    <collision>
-      <origin xyz="-0.01 0 -0.785" rpy="1.57 0 -1.57" />
-      <geometry>
-        <mesh filename="package://thesis_robot_modeling/meshes/lidar_link.STL" />
-      </geometry>
-    </collision>
-  </link>
   <joint name="realsense_joint" type="fixed">
     <origin xyz="0.079 0.001 0.285" rpy="-1.57 0 -1.57" />

Commit message: nothing

File: thesis_robot_modeling/urdf/thesis_robot_modeling.urdf.xacro (robot description, xacro)
@@ -144,4 +144,37 @@
     </collision>
   </link>
+  <joint name="rplidar_joint" type="fixed">
+    <origin xyz="-0.01 0 0.335" rpy="0 0 3.14" />
+    <parent link="base_link" />
+    <child link="lidar_link" />
+  </joint>
+  <link name="lidar_link">
+    <inertial>
+      <origin xyz="0 0 0" rpy="0 0 0" />
+      <mass value="0.021237" />
+      <inertia
+        ixx="0.00016144"
+        ixy="2.1931E-07"
+        ixz="-4.8964E-07"
+        iyy="0.00020117"
+        iyz="-2.029E-05"
+        izz="0.00010111" />
+    </inertial>
+    <visual>
+      <origin xyz="-0.01 0 -0.785" rpy="1.57 0 -1.57" />
+      <geometry>
+        <mesh filename="package://thesis_robot_modeling/meshes/lidar_link.STL" />
+      </geometry>
+      <material name="">
+        <color rgba="0.79216 0.81961 0.93333 1" />
+      </material>
+    </visual>
+    <collision>
+      <origin xyz="-0.01 0 -0.785" rpy="1.57 0 -1.57" />
+      <geometry>
+        <mesh filename="package://thesis_robot_modeling/meshes/lidar_link.STL" />
+      </geometry>
+    </collision>
+  </link>
   <joint name="realsense_joint" type="fixed">
     <origin xyz="0.079 0.001 0.285" rpy="-1.57 0 -1.57" />
